Commit message: Fix the leg.xacro

File: unitree_go2_description/urdf/leg.xacro (robot description, xacro)
@@ -128,5 +128,5 @@
             </inertial>
         </link>
-        <joint name="${name}_foot_joint" type="fixed">0
+        <joint name="${name}_foot_joint" type="fixed">
             <origin rpy="0 0 0" xyz="0 0 ${-(calf_length)}"/>
             <parent link="${name}_lower_leg_link"/>
