Commit message: Add comprehensive Go2 namespace support for multi-robot simulation
- Implemented namespace support across all URDF/Xacro files
- Added conditional namespace prefixing to all links and joints
- Created dual robot state publishers (global and namespaced)
- Developed combined controller configuration system
- Added dedicated go2_1 launch file with shared RViz visualization
- Comprehensive multi-robot setup documentation

Features:
- Multi-robot spawning with namespace isolation
- Proper TF tree separation for each robot
- Controller configuration for both robots
- EKF localization with namespace support
- Shared visualization in single RViz instance

Known limitation: Gazebo ros2_control only supports one robot's hardware interfaces

🤖 Generated with [Claude Code](https://claude.ai/code)

Co-Authored-By: Claude <noreply@anthropic.com>

File: unitree_go2_description/urdf/leg.xacro (robot description, xacro)
@@ -3,5 +3,5 @@
     <!-- <xacro:include filename="$(find unitree_go2_description)/transmission.xacro"/> -->
     <xacro:macro name="leg" params="name mirror mirror_dae front_hind front_hind_dae">
-        <joint name="${name}_hip_joint" type="revolute">
+        <joint name="${ns_prefix}${name}_hip_joint" type="revolute">
             <xacro:if value="${(mirror_dae == False) and (front_hind_dae == True)}">
                 <origin rpy="0 0 0" xyz="${leg_offset_x} ${-leg_offset_y} 0"/>
@@ -16,6 +16,6 @@
                 <origin rpy="0 0 0" xyz="${-leg_offset_x} ${leg_offset_y} 0"/>
             </xacro:if>
-            <parent link="trunk"/>
-            <child link="${name}_hip_link"/>
+            <parent link="${ns_prefix}trunk"/>
+            <child link="${ns_prefix}${name}_hip_link"/>
             <axis xyz="1 0 0"/>
             <dynamics damping="${damping}" friction="${friction}"/>
@@ -27,5 +27,5 @@
             </xacro:if>
         </joint>
-        <link name="${name}_hip_link">
+        <link name="${ns_prefix}${name}_hip_link">
             <visual>
                 <xacro:if value="${(mirror_dae == True) and (front_hind_dae == True)}">
@@ -61,13 +61,13 @@
             </inertial>
         </link>
-        <joint name="${name}_upper_leg_joint" type="revolute">
+        <joint name="${ns_prefix}${name}_upper_leg_joint" type="revolute">
             <origin rpy="0 0 0" xyz="0 ${thigh_offset*mirror} 0"/>
-            <parent link="${name}_hip_link"/>
-            <child link="${name}_upper_leg_link"/>
+            <parent link="${ns_prefix}${name}_hip_link"/>
+            <child link="${ns_prefix}${name}_upper_leg_link"/>
             <axis xyz="0 1 0"/>
             <dynamics damping="${damping}" friction="${friction}"/>
             <limit effort="${thigh_torque_max}" velocity="${thigh_velocity_max}" lower="${thigh_position_min}" upper="${thigh_position_max}"/>
         </joint>
-        <link name="${name}_upper_leg_link">
+        <link name="${ns_prefix}${name}_upper_leg_link">
             <visual>
                 <origin rpy="0 0 0" xyz="0 0 0"/>
@@ -97,13 +97,13 @@
             </inertial>
         </link>
-        <joint name="${name}_lower_leg_joint" type="revolute">
+        <joint name="${ns_prefix}${name}_lower_leg_joint" type="revolute">
             <origin rpy="0 0 0" xyz="0 0 ${-thigh_length}"/>
-            <parent link="${name}_upper_leg_link"/>
-            <child link="${name}_lower_leg_link"/>
+            <parent link="${ns_prefix}${name}_upper_leg_link"/>
+            <child link="${ns_prefix}${name}_lower_leg_link"/>
             <axis xyz="0 1 0"/>
             <dynamics damping="${damping}" friction="${friction}"/>
             <limit effort="${calf_torque_max}" velocity="${calf_velocity_max}" lower="${calf_position_min}" upper="${calf_position_max}"/>
         </joint>
-        <link name="${name}_lower_leg_link">
+        <link name="${ns_prefix}${name}_lower_leg_link">
             <visual>
                 <origin rpy="0 0 0" xyz="0 0 0"/>
@@ -128,10 +128,10 @@
             </inertial>
         </link>
-        <joint name="${name}_foot_joint" type="fixed">0
+        <joint name="${ns_prefix}${name}_foot_joint" type="fixed">
             <origin rpy="0 0 0" xyz="0 0 ${-(calf_length)}"/>
-            <parent link="${name}_lower_leg_link"/>
-            <child link="${name}_foot_link"/>
+            <parent link="${ns_prefix}${name}_lower_leg_link"/>
+            <child link="${ns_prefix}${name}_foot_link"/>
         </joint>
-        <link name="${name}_foot_link">
+        <link name="${ns_prefix}${name}_foot_link">
             <visual>
                 <origin rpy="0 0 0" xyz="0 0 0"/>
@@ -159,15 +159,15 @@
                 <plugin>gz_ros2_control/GazeboSimSystem</plugin>
             </hardware>
-            <joint name="${name}_hip_joint">
+            <joint name="${ns_prefix}${name}_hip_joint">
                 <command_interface name="effort"/>
                 <state_interface name="position"/>
                 <state_interface name="velocity"/>
             </joint>
-            <joint name="${name}_upper_leg_joint">
+            <joint name="${ns_prefix}${name}_upper_leg_joint">
                 <command_interface name="effort"/>
                 <state_interface name="position"/>
                 <state_interface name="velocity"/>
             </joint>
-            <joint name="${name}_lower_leg_joint">
+            <joint name="${ns_prefix}${name}_lower_leg_joint">
                 <command_interface name="effort"/>
                 <state_interface name="position"/>

File: unitree_go2_description/urdf/lidar_4D_lidar.xacro (robot description, xacro)
@@ -2,5 +2,5 @@
 <robot xmlns:xacro="http://www.ros.org/wiki/xacro">
     <!-- Lidar L1-->
-    <link name="lidar_l1_link">
+    <link name="${ns_prefix}lidar_l1_link">
         <inertial>
             <mass value="0.5"/>
@@ -28,10 +28,10 @@
     </link>
     <joint name="lidar_l1_joint" type="fixed">
-        <parent link="base_link"/>
-        <child link="lidar_l1_link"/>
+        <parent link="${ns_prefix}base_link"/>
+        <child link="${ns_prefix}lidar_l1_link"/>
         <!-- <origin rpy="2.94 0 1.5705" xyz="0.25 -0.038 -0.03"/> -->
         <origin rpy="2.879 0.0 1.5705" xyz="0.25 -0.038 -0.03"/>
     </joint>
-    <gazebo reference="lidar_l1_link">
+    <gazebo reference="${ns_prefix}lidar_l1_link">
         <sensor name="lidar_l1" type="gpu_lidar">
             <topic>unitree_lidar</topic>
@@ -64,5 +64,5 @@
             </lidar>
             <visualize>false</visualize>
-            <gz_frame_id>lidar_l1_link</gz_frame_id>
+            <gz_frame_id>${ns_prefix}lidar_l1_link</gz_frame_id>
             <always_on>1</always_on>
         </sensor>

File: unitree_go2_description/urdf/unitree_go2_gazebo.xacro (robot description, xacro)
@@ -1,4 +1,4 @@
 <?xml version="1.0"?>
-<robot>
+<robot xmlns:xacro="http://www.ros.org/wiki/xacro">
   <!-- Gazebo Sim plugins -->
   <gazebo>
@@ -25,5 +25,5 @@
   <gazebo>
     <plugin filename="gz_ros2_control-system" name="gz_ros2_control::GazeboSimROS2ControlPlugin">
-      <parameters>$(find unitree_go2_sim)/config/ros_control/ros_control.yaml</parameters>
+      <parameters>${ros_control_config_file if ros_control_config_file else '$(find unitree_go2_sim)/config/ros_control/ros_control.yaml'}</parameters>
       <robot_param_node>robot_state_publisher</robot_param_node>
     </plugin>
@@ -33,5 +33,5 @@
     <plugin filename="gz-sim-odometry-publisher-system" name="gz::sim::systems::OdometryPublisher">
       <odom_frame>odom</odom_frame>
-      <robot_base_frame>base_link</robot_base_frame>
+      <robot_base_frame>${ns_prefix}base_link</robot_base_frame>
       <odom_topic>/odom</odom_topic>
       <odom_publish_frequency>50</odom_publish_frequency>
@@ -39,5 +39,5 @@
   </gazebo>
   <!-- IMU plugin -->
-  <gazebo reference="imu_link">
+  <gazebo reference="${ns_prefix}imu_link">
     <sensor name="imu_sensor" type="imu">
       <always_on>true</always_on>
@@ -45,5 +45,5 @@
       <visualize>true</visualize>
       <topic>imu/data</topic>
-      <gz_frame_id>imu_link</gz_frame_id>
+      <gz_frame_id>${ns_prefix}imu_link</gz_frame_id>
       <imu>
         <angular_velocity>
@@ -94,5 +94,5 @@
   </gazebo>
   <!-- Camera Plugin-->
-  <gazebo reference="camera_link">
+  <gazebo reference="${ns_prefix}camera_link">
     <sensor name="rgb_camera" type="camera">
       <pose>0 0.0 0 0 0 0</pose>
@@ -108,5 +108,5 @@
         </clip>
       </camera>
-      <gz_frame_id>camera_link</gz_frame_id>
+      <gz_frame_id>${ns_prefix}camera_link</gz_frame_id>
       <always_on>1</always_on>
       <update_rate>10</update_rate>
@@ -116,5 +116,5 @@
   </gazebo>
   <!-- Main body -->
-  <gazebo reference="trunk">
+  <gazebo reference="${ns_prefix}trunk">
     <mu1>0.2</mu1>
     <mu2>0.2</mu2>
@@ -123,21 +123,21 @@
   </gazebo>
   <!-- FL leg -->
-  <gazebo reference="lf_hip_link">
-    <mu1>0.2</mu1>
-    <mu2>0.2</mu2>
-  </gazebo>
-  <gazebo reference="lf_upper_leg_link">
-    <mu1>0.2</mu1>
-    <mu2>0.2</mu2>
-    <self_collide>1</self_collide>
-    <kp>10000.0</kp>
-    <kd>1.0</kd>
-  </gazebo>
-  <gazebo reference="lf_lower_leg_link">
-    <mu1>0.2</mu1>
-    <mu2>0.2</mu2>
-    <self_collide>1</self_collide>
-  </gazebo>
-  <gazebo reference="lf_foot_link">
+  <gazebo reference="${ns_prefix}lf_hip_link">
+    <mu1>0.2</mu1>
+    <mu2>0.2</mu2>
+  </gazebo>
+  <gazebo reference="${ns_prefix}lf_upper_leg_link">
+    <mu1>0.2</mu1>
+    <mu2>0.2</mu2>
+    <self_collide>1</self_collide>
+    <kp>10000.0</kp>
+    <kd>1.0</kd>
+  </gazebo>
+  <gazebo reference="${ns_prefix}lf_lower_leg_link">
+    <mu1>0.2</mu1>
+    <mu2>0.2</mu2>
+    <self_collide>1</self_collide>
+  </gazebo>
+  <gazebo reference="${ns_prefix}lf_foot_link">
     <mu1>0.6</mu1>
     <mu2>0.6</mu2>
@@ -147,21 +147,21 @@
   </gazebo>
   <!-- FR leg -->
-  <gazebo reference="rf_hip_link">
-    <mu1>0.2</mu1>
-    <mu2>0.2</mu2>
-  </gazebo>
-  <gazebo reference="rf_upper_leg_link">
-    <mu1>0.2</mu1>
-    <mu2>0.2</mu2>
-    <self_collide>1</self_collide>
-    <kp>10000.0</kp>
-    <kd>1.0</kd>
-  </gazebo>
-  <gazebo reference="rf_lower_leg_link">
-    <mu1>0.2</mu1>
-    <mu2>0.2</mu2>
-    <self_collide>1</self_collide>
-  </gazebo>
-  <gazebo reference="rf_foot_link">
+  <gazebo reference="${ns_prefix}rf_hip_link">
+    <mu1>0.2</mu1>
+    <mu2>0.2</mu2>
+  </gazebo>
+  <gazebo reference="${ns_prefix}rf_upper_leg_link">
+    <mu1>0.2</mu1>
+    <mu2>0.2</mu2>
+    <self_collide>1</self_collide>
+    <kp>10000.0</kp>
+    <kd>1.0</kd>
+  </gazebo>
+  <gazebo reference="${ns_prefix}rf_lower_leg_link">
+    <mu1>0.2</mu1>
+    <mu2>0.2</mu2>
+    <self_collide>1</self_collide>
+  </gazebo>
+  <gazebo reference="${ns_prefix}rf_foot_link">
     <mu1>0.6</mu1>
     <mu2>0.6</mu2>
@@ -171,21 +171,21 @@
   </gazebo>
   <!-- RL leg -->
-  <gazebo reference="lh_hip_link">
-    <mu1>0.2</mu1>
-    <mu2>0.2</mu2>
-  </gazebo>
-  <gazebo reference="lh_upper_leg_link">
-    <mu1>0.2</mu1>
-    <mu2>0.2</mu2>
-    <self_collide>1</self_collide>
-    <kp>10000.0</kp>
-    <kd>1.0</kd>
-  </gazebo>
-  <gazebo reference="lh_lower_leg_link">
-    <mu1>0.2</mu1>
-    <mu2>0.2</mu2>
-    <self_collide>1</self_collide>
-  </gazebo>
-  <gazebo reference="lh_foot_link">
+  <gazebo reference="${ns_prefix}lh_hip_link">
+    <mu1>0.2</mu1>
+    <mu2>0.2</mu2>
+  </gazebo>
+  <gazebo reference="${ns_prefix}lh_upper_leg_link">
+    <mu1>0.2</mu1>
+    <mu2>0.2</mu2>
+    <self_collide>1</self_collide>
+    <kp>10000.0</kp>
+    <kd>1.0</kd>
+  </gazebo>
+  <gazebo reference="${ns_prefix}lh_lower_leg_link">
+    <mu1>0.2</mu1>
+    <mu2>0.2</mu2>
+    <self_collide>1</self_collide>
+  </gazebo>
+  <gazebo reference="${ns_prefix}lh_foot_link">
     <mu1>0.6</mu1>
     <mu2>0.6</mu2>
@@ -195,21 +195,21 @@
   </gazebo>
   <!-- RR leg -->
-  <gazebo reference="rh_hip_link">
-    <mu1>0.2</mu1>
-    <mu2>0.2</mu2>
-  </gazebo>
-  <gazebo reference="rh_upper_leg_link">
-    <mu1>0.2</mu1>
-    <mu2>0.2</mu2>
-    <self_collide>1</self_collide>
-    <kp>10000.0</kp>
-    <kd>1.0</kd>
-  </gazebo>
-  <gazebo reference="rh_lower_leg_link">
-    <mu1>0.2</mu1>
-    <mu2>0.2</mu2>
-    <self_collide>1</self_collide>
-  </gazebo>
-  <gazebo reference="rh_foot_link">
+  <gazebo reference="${ns_prefix}rh_hip_link">
+    <mu1>0.2</mu1>
+    <mu2>0.2</mu2>
+  </gazebo>
+  <gazebo reference="${ns_prefix}rh_upper_leg_link">
+    <mu1>0.2</mu1>
+    <mu2>0.2</mu2>
+    <self_collide>1</self_collide>
+    <kp>10000.0</kp>
+    <kd>1.0</kd>
+  </gazebo>
+  <gazebo reference="${ns_prefix}rh_lower_leg_link">
+    <mu1>0.2</mu1>
+    <mu2>0.2</mu2>
+    <self_collide>1</self_collide>
+  </gazebo>
+  <gazebo reference="${ns_prefix}rh_foot_link">
     <mu1>0.6</mu1>
     <mu2>0.6</mu2>

File: unitree_go2_description/urdf/unitree_go2_robot.xacro (robot description, xacro)
@@ -3,4 +3,9 @@
     xmlns:xacro="http://www.ros.org/wiki/xacro">
     <xacro:arg name="DEBUG" default="false"/>
+    <xacro:arg name="namespace" default=""/>
+    <xacro:arg name="ros_control_config_file" default=""/>
+    <!-- Create namespace prefix property -->
+    <xacro:property name="ns_prefix" value="${'$(arg namespace)/' if '$(arg namespace)' != '' else ''}" />
+    <xacro:property name="ros_control_config_file" value="$(arg ros_control_config_file)" />
     <xacro:include filename="$(find unitree_go2_description)/urdf/const.xacro"/>
     <xacro:include filename="$(find unitree_go2_description)/urdf/materials.xacro"/>
@@ -20,8 +25,8 @@
             <origin rpy="0 0 0" xyz="0 0 0"/>
             <parent link="world"/>
-            <child link="base_link"/>
+            <child link="${ns_prefix}base_link"/>
         </joint>
     </xacro:if>
-    <link name="base_link">
+    <link name="${ns_prefix}base_link">
         <visual>
             <origin rpy="0 0 0" xyz="0 0 0"/>
@@ -33,8 +38,8 @@
     <joint name="floating_base" type="fixed">
         <origin rpy="0 0 0" xyz="0 0 0"/>
-        <parent link="base_link"/>
-        <child link="trunk"/>
+        <parent link="${ns_prefix}base_link"/>
+        <child link="${ns_prefix}trunk"/>
     </joint>
-    <link name="trunk">
+    <link name="${ns_prefix}trunk">
         <visual>
             <origin rpy="0 0 0" xyz="0 0 0"/>
@@ -56,9 +61,9 @@
     </link>
     <joint name="imu_joint" type="fixed">
-        <parent link="trunk"/>
-        <child link="imu_link"/>
+        <parent link="${ns_prefix}trunk"/>
+        <child link="${ns_prefix}imu_link"/>
         <origin rpy="0 0 0" xyz="0 0 0"/>
     </joint>
-    <link name="imu_link">
+    <link name="${ns_prefix}imu_link">
         <inertial>
             <mass value="0.001"/>
@@ -80,5 +85,5 @@
     </link>
     <!-- Camera Link-->
-    <link name="camera_link">
+    <link name="${ns_prefix}camera_link">
         <inertial>
             <mass value="0.001"/>
@@ -103,6 +108,6 @@
     </link>
     <joint name="camera_joint" type="fixed">
-        <parent link="trunk"/>
-        <child link="camera_link"/>
+        <parent link="${ns_prefix}trunk"/>
+        <child link="${ns_prefix}camera_link"/>
         <origin rpy="0 0 0" xyz="0.326 0 0.043"/>
     </joint>

File: unitree_go2_description/urdf/velodyne.xacro (robot description, xacro)
@@ -3,8 +3,8 @@
     <joint name="velodyne_base_mount_joint" type="fixed">
         <origin rpy="0 0 0" xyz="0.2 0 0.08"/>
-        <parent link="base_link"/>
-        <child link="velodyne_base_link"/>
+        <parent link="${ns_prefix}base_link"/>
+        <child link="${ns_prefix}velodyne_base_link"/>
     </joint>
-    <link name="velodyne_base_link">
+    <link name="${ns_prefix}velodyne_base_link">
         <inertial>
             <mass value="0.83"/>
@@ -31,8 +31,8 @@
     <joint name="velodyne_base_scan_joint" type="fixed">
         <origin rpy="0 0 0" xyz="0 0 0.0377"/>
-        <parent link="velodyne_base_link"/>
-        <child link="velodyne"/>
+        <parent link="${ns_prefix}velodyne_base_link"/>
+        <child link="${ns_prefix}velodyne"/>
     </joint>
-    <link name="velodyne">
+    <link name="${ns_prefix}velodyne">
         <inertial>
             <mass value="0.01"/>
@@ -48,9 +48,9 @@
     </link>
     <!-- Gazebo Sim Velodyne Sensor plugin -->
-    <gazebo reference="velodyne">
+    <gazebo reference="${ns_prefix}velodyne">
         <sensor name="velodyne-VLP16" type="gpu_lidar">
             <topic>velodyne_points</topic>
             <update_rate>10</update_rate>
-            <gz_frame_id>velodyne</gz_frame_id>
+            <gz_frame_id>${ns_prefix}velodyne</gz_frame_id>
             <lidar>
                 <scan>
@@ -78,5 +78,5 @@
                     <stddev>0.008</stddev>
                 </noise>
-                <frame_id>velodyne</frame_id>
+                <frame_id>${ns_prefix}velodyne</frame_id>
             </lidar>
             <visualize>true</visualize>
